File: panel/VCO-Simple-Panel.vC.kicad_pcb (KiCad board)
At the start: 2 copper layers, 30.5 x 128.2 mm, 1 part

Commit message: panel updates
Parts:
- added G***: LOGO, artwork:F.Cu_g17, F.Cu at (148.6, 113.0)
Routing:
- removed copper zone on F.Cu, net (none)
